File: pcb/KiCAD/VORTAC_TOOLPLATE_REV1/VORTAC_TOOLPLATE_REV1.kicad_pcb (KiCad board)
At the start: 4 copper layers, 15.4 x 24 mm, 10 parts, among them J1 Conn_01x07, J2 Conn_01x02, J3 Conn_01x05

Commit message: Added Dock PCB
Connections:
- D1 pad 2: CAN_H -> CAN_L
- D2 pad 2: CAN_L -> CAN_H
- J1 pad 6: CAN_H -> CAN_L
- J1 pad 7: CAN_L -> CAN_H
- J3 pad 4: CAN_H -> CAN_L
- J3 pad 5: CAN_L -> CAN_H
