File: pcb/KiCAD/VORTAC_DOCK_REV1/VORTAC_DOCK_REV1.kicad_pcb (KiCad board)
At the start: 4 copper layers, 24.8 x 17.6 mm, 27 parts, among them J1 Conn_01x01, J2 Conn_01x01, J3 Conn_01x05, J4 Conn_01x03, J5 Conn_01x03, U1 AP63205WU, U2 WS2811, U3 TPS26630RGE

Commit message: Doc Rev1 revision
Parts:
- added C34: 100uF 35V, Capacitor_SMD:CP_Elec_6.3x7.7, F.Cu at (100.2, 108.0)
- added D5: PTVS26VS1UR,115-ES, Diode_SMD:D_SOD-123F, F.Cu at (100.0, 117.6)
- U2: footprint Package_TO_SOT_SMD:SOT-23-8 -> Vortac:SOT-23-8; 8mm pitch
- moved J1 4.00 mm to (100.0, 102.5)
- moved R7 0.46 mm to (91.5, 117.5)
- moved U2 0.24 mm to (92.5, 120.0)
Routing:
- net VDC: track 3.65 -> 6.78 mm, vias 6 -> 10
- net GND: vias 31 -> 34
Other:
- board size 24.8 x 17.6 mm -> 24.8 x 21.6 mm
- board text added: "VORTAC"
